File: PCB/RP2354A_Cluster/RP2354A_Cluster.kicad_pcb (KiCad board)
At the start: 4 copper layers, 43 x 24.8 mm, 114 parts, among them SW1 miniButton, SW2 miniButton, U13 SL2.1A, U14 USB, U15 TPS62933, U16 TPS62933, U17 RP2340, U18 RP2340, U19 RP2340, U20 RP2340, Y1 12MHz GND24, Y2 12MHz GND24, Y3 12MHz GND24, Y4 12MHz GND24, Y5 12MHz GND24

Commit message: fixed power stuff
Parts:
- removed Y5: 12MHz GND24, Crystal:Crystal_SMD_2520-4Pin_2.5x2.0mm
- added C78: 4.7u, Basics:C_0402_1005Metric, F.Cu at (103.8, 66.9)
- added C79: 4.7u, Basics:C_0402_1005Metric, F.Cu at (107.5, 72.8)
- added C80: 4.7u, Basics:C_0402_1005Metric, F.Cu at (113.3, 69.0)
- added C81: 4.7u, Basics:C_0402_1005Metric, F.Cu at (109.5, 63.2)
- R27: value 31.3 -> 31.3k
- moved R9 0.15 mm to (106.3, 71.6)
- moved R19 0.14 mm to (110.7, 64.4)
- moved R2 0.14 mm to (104.9, 65.8)
- moved R14 0.13 mm to (112.1, 70.2)
Connections:
- U13 pad 15: Net-(U13-XOUT) -> unconnected-(U13-XOUT-Pad15)
- U13 pad 16: Net-(U13-XIN) -> GND
- U17 pad 46: unconnected-(U17-VREG_AVDD-Pad46) -> +3.3V
- U17 pad 47: unconnected-(U17-VREG_PGND-Pad47) -> GND
- U17 pad 49: unconnected-(U17-VREG_VIN-Pad49) -> +3.3V
- U17 pad 50: unconnected-(U17-VREG_FB-Pad50) -> GND
- U18 pad 46: unconnected-(U18-VREG_AVDD-Pad46) -> +3.3V
- U18 pad 47: unconnected-(U18-VREG_PGND-Pad47) -> GND
- U18 pad 49: unconnected-(U18-VREG_VIN-Pad49) -> +3.3V
- U18 pad 50: unconnected-(U18-VREG_FB-Pad50) -> GND
- U19 pad 46: unconnected-(U19-VREG_AVDD-Pad46) -> +3.3V
- U19 pad 47: unconnected-(U19-VREG_PGND-Pad47) -> GND
- U19 pad 49: unconnected-(U19-VREG_VIN-Pad49) -> +3.3V
- U19 pad 50: unconnected-(U19-VREG_FB-Pad50) -> GND
- U20 pad 46: unconnected-(U20-VREG_AVDD-Pad46) -> +3.3V
- U20 pad 47: unconnected-(U20-VREG_PGND-Pad47) -> GND
- U20 pad 49: unconnected-(U20-VREG_VIN-Pad49) -> +3.3V
- U20 pad 50: unconnected-(U20-VREG_FB-Pad50) -> GND
Routing:
- net +3.3V: track 270.2 -> 283.9 mm
- net Net-(U13-XOUT): track 4.28 -> 0.00 mm
- net Net-(U13-XIN): track 3.48 -> 0.00 mm
- net GND: vias 120 -> 123
